File: rtcl-ae-ft232hl-jtag/rtcl-ae-ft232hl-jtag.kicad_pcb (KiCad board)
At the start: 2 copper layers, 20.3 x 52.1 mm, 3 parts, among them J1 Conn_01x14, J2 Conn_01x14, J3 Conn_01x06

Commit message: WIP
Parts:
- J3: footprint Connector_PinSocket_2.54mm:PinSocket_1x06_P2.54mm_Horizontal -> rtcl-ae-ft232hl-jtag:PinSocket_1x06_P2.54mm_Horizontal
Routing:
- net /TCK: track 29.1 -> 46.8 mm
- net /TDI: track 24.4 -> 37.7 mm
- net GND: track 80.9 -> 92.6 mm
- net /TDO: track 29.6 -> 37.7 mm
- net /TMS: track 19.4 -> 24.5 mm
- net VDD: track 43.9 -> 40.3 mm
Other:
- board text added: "GND"
- board text added: "TCK"
- board text added: "TDI"
- board text added: "TDO"
- board text added: "TMS"
- board text added: "VDD"
