File: rtcl-ae-ft232hl-jtag/rtcl-ae-ft232hl-jtag.kicad_sch (KiCad schematic)
At the start: 3 parts, among them J1 Conn_01x14, J2 Conn_01x14, J3 Conn_01x06

Commit message: WIP
Parts:
- J3: footprint Connector_PinSocket_2.54mm:PinSocket_1x06_P2.54mm_Horizontal -> rtcl-ae-ft232hl-jtag:PinSocket_1x06_P2.54mm_Horizontal
Changed lines of the file:
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@@
 			)
 		)
-		(property "Footprint" "Connector_PinSocket_2.54mm:PinSocket_1x06_P2.54mm_Horizontal"
+		(property "Footprint" "rtcl-ae-ft232hl-jtag:PinSocket_1x06_P2.54mm_Horizontal"
 			(at 171.45 67.31 0)
 			(hide yes)
